File: SDR intro/SDR intro.kicad_pcb (KiCad board)
At the start: 4 copper layers, 75 x 25 mm, 59 parts, among them J1 3220-20-0200-00, J2 GSB1C41110SSHR, J3 1984617, J4 647676-2, Q1 NMOS, U1 LMH6702MF, U3 SST25VF010A-33-4C-SAE-T, U5 BMP390, U6 CP2102N-A02-GQFN20, U7 STM32G441KBT6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

Commit message: d
Parts:
- removed D5, D6: D, Diode_SMD:D_0603_1608Metric
- added C3: .1 uF, Capacitor_SMD:C_0603_1608Metric, F.Cu at (103.7, 99.8)
- added CR2: UFM15PL-TP, pretty diode:SOD-123FL_MCC, F.Cu at (73.5, 101.6)
- added CR3: UFM15PL-TP, pretty diode:SOD-123FL_MCC, F.Cu at (70.7, 100.6)
- added JP1: Jumper_2_Open, Resistor_SMD:R_0603_1608Metric, F.Cu at (55.6, 108.7)
- added JP2: Jumper_2_Open, Resistor_SMD:R_0603_1608Metric, F.Cu at (76.2, 92.5)
- added S1: 435171014816, 435171014816:435171014816, F.Cu at (73.0, 92.2)
- C14: value 100 uF -> 100 nF
- C16: value 120 uF -> 120 nF
- R8, R9: value R -> 100 k
- moved R19 13.1 mm to (87.3, 95.5), turned to -90 degrees
Connections:
- U6 pad 17: UART_RXD -> UART_TXD
- U6 pad 18: UART_TXD -> UART_RXD
- U7 pad 31: unconnected-(U7A-PB8-BOOT0-Pad31) -> Boot
Routing:
- net Boot: track 0.00 -> 47.3 mm, vias 0 -> 4
- net NRST: track 33.9 -> 71.1 mm, vias 2 -> 6
- net 5V: track 79.1 -> 100.5 mm, vias 6 -> 8
- net +3.3V: track 73.7 -> 69.0 mm
- net BNO_SDA: track 51.2 -> 55.1 mm
- net GND: track 87.1 -> 90.9 mm, vias 30 -> 31
- net Net-(JP2-B): track 0.00 -> 2.07 mm
- net Battery: track 61.9 -> 63.0 mm
- net PRD_SWO: track 28.2 -> 29.0 mm
- net SWITCH: track 32.1 -> 32.6 mm
