File: SDR intro/SDR intro.kicad_sch (KiCad schematic)
At the start: 59 parts, among them J1 3220-20-0200-00, J2 GSB1C41110SSHR, J3 1984617, J4 647676-2, Q1 NMOS, U1 LMH6702MF, U3 SST25VF010A-33-4C-SAE-T, U5 BMP390, U6 CP2102N-A02-GQFN20, U7 STM32G441KBT6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

Commit message: d
Parts:
- removed D5, D6: D, Diode_SMD:D_0603_1608Metric, symbol Device:D
- added C3: .1 uF, Capacitor_SMD:C_0603_1608Metric, symbol Device:C
- added CR2, CR3: UFM15PL-TP, pretty diode:SOD-123FL_MCC, symbol Friendly diode:UFM15PL-TP
- added JP1, JP2: Jumper_2_Open, Resistor_SMD:R_0603_1608Metric, symbol Jumper:Jumper_2_Open
- added S1: 435171014816, 435171014816:435171014816, symbol 435171014816:435171014816
- C10, C2: value 0.1up -> 0.1uF
- C11: value 1 -> 1 uF
- C14: value 100 uF -> 100 nF
- C16: value 120 uF -> 120 nF
- C17: value 10 -> 10 uF
- C18, C20: value .1 -> .1 uF
- C19: value 4.7 -> 4.7 uF
- R8, R9: value R -> 100 k
Connections:
- net +3.3V: now also JP1.1 (A)
- net 5V: now also CR3.2
- net Battery: now also CR2.2
- net GND: now also C3.2, JP2.1 (A)
- net NRST: now also C3.1, S1.1
- net UART_RXD: now also U6.18 (TXD); no longer U6.17 (RXD)
- net UART_TXD: now also U6.17 (RXD); no longer U6.18 (TXD)
- net at C13.1, U8.3 (IN): now also CR2.1, CR3.1
- net Boot: now reaches U7.31 (PB8-BOOT0)
- net Boot: now also JP1.2 (B)
- new net: JP2.2 (B), S1.3
- no-connect marks 21 -> 25
Other:
- moved on the sheet: C14, C15, C16, D1, H1, H2, H3, H4, R17, R18, R19, R3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
